File: Power_Control_Unit_PCB.kicad_sch (KiCad schematic)
At the start: 0 parts

Commit message: PCU Schematics
Parts:
- added C1, C2, C3: 47µ/50V, Capacitor_SMD:CP_Elec_6.3x7.7, symbol BLESS:C_Polarized_47µF
- added C4, C5, C6: 22µ/16V, Capacitor_SMD:CP_Elec_5x5.8, symbol BLESS:C_Polarized_22µF
- added D1, D2, D3: SS36-E3/9AT, Diode_SMD:D_SMC, symbol Diode:SS36
- added F1: 1.25A, Fuse:Fuse_Littelfuse-NANO2-451_453, symbol BLESS:Fuse_Small_1.25A
- added FID1, FID2, FID3: Fiducial, Fiducial:Fiducial_1mm_Mask2mm, symbol Mechanical:Fiducial
- added J1: Molex_Conn_01x04, Connector_Molex:Molex_Micro-Fit_3.0_43650-0415_1x04_P3.00mm_Vertical, symbol BLESS:Molex_Conn_01x04
- added J2: WR-BHD_Conn_02x08_Odd_Even, Connector_IDC:IDC-Header_2x08_P2.54mm_Vertical, symbol BLESS:WR_Conn_02x08
- added J3: WR-BHD_Conn_02x04_Odd_Even, Connector_IDC:IDC-Header_2x04_P2.54mm_Vertical, symbol Connector_Generic:Conn_02x04_Odd_Even
- added J4: WR-BHD_Conn_02x03_Odd_Even, Connector_IDC:IDC-Header_2x03_P2.54mm_Vertical, symbol BLESS:WR-BHD_Conn_02x03_Odd_Even
- added J5: WR-BHD_Conn_02x17_Odd_Even, Connector_IDC:IDC-Header_2x17_P2.54mm_Vertical, symbol Connector_Generic:Conn_02x17_Odd_Even
- added MH1, MH2, MH3, MH4: M3, MountingHole:MountingHole_3.2mm_M3_Pad_Via, symbol Mechanical:MountingHole_Pad
- added U1: TSR_1-2433, Converter_DCDC:Converter_DCDC_TRACO_TSR-1_THT, symbol Converter_DCDC:TSR_1-2433
- added U2: TSR_1-2450, Converter_DCDC:Converter_DCDC_TRACO_TSR-1_THT, symbol Converter_DCDC:TSR_1-2450
- added U3: TSR3-24120N, Converter_DCDC:Converter_DCDC_TRACO_TSR2-24xxN_TSR2-24xxxN_THT, symbol BLESS:TSR3-24120N
Connections:
- new net: C1.1, D1.1 (K), U1.1 (Vin)
- new net: C2.1, D2.1 (K), U2.1 (Vin)
- new net: D1.2 (A), D2.2 (A), D3.2 (A), F1.2
- new net: C3.1, D3.1 (K), U3.1 (Vin)
- new net +12V: C6.1, J4.1 (Pin_1), J4.2 (Pin_2), J4.3 (Pin_3), J4.4 (Pin_4), J4.5 (Pin_5), J4.6 (Pin_6), U3.3 (Vout)
- new net +28V: F1.1, J1.4 (Pin_4)
- new net +3V3: C4.1, J2.1 (Pin_1), J2.10 (Pin_10), J2.11 (Pin_11), J2.12 (Pin_12), J2.13 (Pin_13), J2.14 (Pin_14), J2.15 (Pin_15), J2.16 (Pin_16), J2.2 (Pin_2), J2.3 (Pin_3), J2.4 (Pin_4), J2.5 (Pin_5), J2.6 (Pin_6), J2.7 (Pin_7), J2.8 (Pin_8), J2.9 (Pin_9), U1.3 (Vout)
- new net +5V: C5.1, J3.1 (Pin_1), J3.2 (Pin_2), J3.3 (Pin_3), J3.4 (Pin_4), J3.5 (Pin_5), J3.6 (Pin_6), J3.7 (Pin_7), J3.8 (Pin_8), U2.3 (Vout)
- new net GND: C1.2, C2.2, C3.2, C4.2, C5.2, C6.2, J1.1 (Pin_1), J5.1 (Pin_1), J5.10 (Pin_10), J5.11 (Pin_11), J5.12 (Pin_12), J5.13 (Pin_13), J5.14 (Pin_14), J5.15 (Pin_15), J5.16 (Pin_16), J5.17 (Pin_17), J5.18 (Pin_18), J5.19 (Pin_19), J5.2 (Pin_2), J5.20 (Pin_20), J5.21 (Pin_21), J5.22 (Pin_22), J5.23 (Pin_23), J5.24 (Pin_24), J5.25 (Pin_25), J5.26 (Pin_26), J5.27 (Pin_27), J5.28 (Pin_28), J5.29 (Pin_29), J5.3 (Pin_3), J5.30 (Pin_30), J5.31 (Pin_31), J5.32 (Pin_32), J5.33 (Pin_33), J5.34 (Pin_34), J5.4 (Pin_4), J5.5 (Pin_5), J5.6 (Pin_6), J5.7 (Pin_7), J5.8 (Pin_8), J5.9 (Pin_9), MH1.1, MH2.1, MH3.1, MH4.1, U1.2 (GND), U2.2 (GND), U3.2 (GND)
- no-connect marks 0 -> 2
Other:
- note added: "Power Supply"
- note added: "TO/FROM AMPHENOL"

Commit message: PCU pcb design and added copper zones por power planes
Parts:
- added TP1, TP2, TP3, TP4, TP5: TestPoint, TestPoint:TestPoint_Pad_D1.0mm, symbol Connector:TestPoint
Connections:
- net +12V: now also TP4.1
- net +28V: now also TP1.1
- net +3V3: now also TP2.1
- net +5V: now also TP3.1
- net GND: now also TP5.1
Other:
- moved on the sheet: J1, J2, J3, J4
